File: IDP Schematic/IDP Schematic.kicad_sch (KiCad schematic)
At the start: 27 parts

Commit message: Added AD7920 symbol
Parts:
- added U?: AD7920, symbol IEP:AD7920
Changed lines of the file:
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@@
+    (pin "")
+  )
+  (symbol (lib_id "IEP:AD7920") (at 212.09 100.33 0) (unit 1)
+    (in_bom yes) (on_board yes) (fields_autoplaced)
+    (property "Reference" "U?" (id 0) (at 212.09 88.9 0))
+    (property "Value" "AD7920" (id 1) (at 212.09 91.44 0))
+    (property "Footprint" "" (id 2) (at 212.09 100.33 0)
+      (effects (font (size 1.27 1.27)) hide)
+    )
+    (property "Datasheet" "" (id 3) (at 212.09 100.33 0)
+      (effects (font (size 1.27 1.27)) hide)
+    )
+    (pin "")
+    (pin "")
+    (pin "")
+    (pin "")
+    (pin "")
     (pin "")
   )
@@
       (reference "U?") (unit 1) (value "HC-SR04") (footprint "")
     )
+    (path "/934dd1a4-3cab-40ee-8112-c49e3513d490"
+      (reference "U?") (unit 1) (value "AD7920") (footprint "")
+    )
     (path "/bad75afc-4b6e-458b-819f-f3bb8e4823ce"
